File: schematics/schematics.sch (KiCad schematic (older format))
At the start: 0 parts

Commit message: some cleanup
Changed lines of the file:
@@
 $EndDescr
 $Sheet
-S 1750 2650 1700 1100
-U 55B90459
-F0 "Stylus" 60
-F1 "stylus.sch" 60
-$EndSheet
-$Sheet
-S 5550 3450 2600 1000
+S 3500 2650 1450 1400
 U 55B9BDE9
 F0 "Main Board" 60
 F1 "mainboard.sch" 60
+F2 "MotorPower" O L 3500 3200 60
+F3 "TopCoverGround" U L 3500 3300 60
+F4 "StylusHeadGround" U L 3500 3800 60
+F5 "HeadLoad" O L 3500 3600 60
+F6 "Tracking" I L 3500 3400 60
+F7 "HeadLoadPower" U L 3500 3500 60
+F8 "SensorPower" U L 3500 3700 60
+F9 "MuteSwitch" O L 3500 2950 60
+F10 "CarriageEncoder" I L 3500 3050 60
+F11 "CarriageStopper" I L 3500 2850 60
+F12 "TrackDetect" I L 3500 2750 60
 $EndSheet
+$Sheet
+S 2150 2650 950  1250
+U 55B90459
+F0 "Top Cover" 60
+F1 "stylus.sch" 60
+F2 "MuteSwitch" I R 3100 2950 60
+F3 "CarriageStopper" O R 3100 2850 60
+F4 "TrackDetect" O R 3100 2750 60
+F5 "CarriageEncoder" O R 3100 3050 60
+F6 "MotorPower" I R 3100 3200 60
+F7 "Tracking" O R 3100 3400 60
+F8 "HeadLoadPower" I R 3100 3500 60
+F9 "SensorPower" I R 3100 3700 60
+F10 "HeadLoad" I R 3100 3600 60
+F11 "TopCoverGround" U R 3100 3300 60
+F12 "StylusHeadGround" U R 3100 3800 60
+$EndSheet
+Wire Wire Line
+	3100 2750 3500 2750
+Wire Wire Line
+	3100 2850 3500 2850
+Wire Wire Line
+	3100 2950 3500 2950
+Wire Wire Line
+	3100 3050 3500 3050
+Wire Wire Line
+	3100 3200 3500 3200
+Wire Wire Line
+	3100 3300 3500 3300
+Wire Wire Line
+	3100 3400 3500 3400
+Wire Wire Line
+	3100 3500 3500 3500
+Wire Wire Line
+	3500 3600 3100 3600
+Wire Wire Line
+	3100 3700 3500 3700
+Wire Wire Line
+	3500 3800 3100 3800
 $EndSCHEMATC
