File: schematics/mainboard.sch (KiCad schematic (older format))
At the start: 88 parts, among them IC1 DIL42, IC2 4069, IC6 RC4558, IC8 LM324N, J108 CONN_01X07, J111 CONN_01X07, J200 CONN_01X04, J55 330k, Q10 2SC1384, Q11 2SC1740S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

Commit message: some cleanup
Parts:
- removed C?: C, symbol C
- removed D10: D, symbol D
- removed R100, R99: R, symbol R
- removed R101: 180k, symbol R
- removed R104: 4k7, symbol R
Connections:
- net labels added: CarriageEncoder, CarriageStopper, ENCODER, HEAD_LOAD, HeadLoad, HeadLoadPower, MUTE, MotorPower, MuteSwitch, PLAY, SensorPower, StylusHeadGround, TopCoverGround, TrackDetect, Tracking, pin33, pin5
- net labels removed: STYLUS_ENGAGE
- wire segments 226 -> 236
- no-connect marks 0 -> 1
Other:
- note added: "???"
- moved on the sheet: C12, C26, C32, C33, D10, D4, D7, D8, D9, IC2C, J108, P?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

Commit message: I think I'm done with track detection circuit
Parts:
- removed C?: VAL, symbol CP1
- removed U? (x2): 4001, symbol 4001
- removed VR4: 100k, symbol POT
- added C42, C? (x2): C, symbol C
- added C43, C?: CP1, symbol CP1
- added D16: D, symbol D
- added unit 2 of IC7
- added unit 3 of IC7
- added unit 1 of IC8
- added unit 2 of IC8
- added J?: CONN_01X04, symbol CONN_01X04
- added Pin_B, Wire_I1: CONN_01X01, symbol CONN_01X01
- added R113, R114, R117, R?: R, symbol R
- added R115: 12k, symbol R
- added R116: 120, symbol R
- added R118?: 47k, symbol R
- added R?: 20k, symbol R
- added R?: 100k, symbol R
- added R?: 150, symbol R
- added R?: 390, symbol R
- added RV4: 100k, symbol POT
- added RV? (x2): 1M, symbol POT
- gave numbers to parts that had none: 2
Connections:
- net GND: now also R121.1, C?.2, D16.2 (A), J?.4 (P4), R113.1, R116.1, R117.1, R118?.2, R?.1, R?.2, RV?.2, RV?.3; no longer R121.2
- net TrackDetect: now also C?.1, IC8.3 (+), RV?.1, RV?.2, RV?.3
- net VCC: now also R119.2, R115.2, R?.2, RV4.2, RV4.3
- net VDD: now also IC7.14 (VDD), IC7.14 (VDD)
- net VSS: now also IC7.7 (VSS), IC7.7 (VSS)
- net pin5: now also R121.2, IC7.6; no longer R121.1
- net at R123.2: now also D15.2 (A), IC7.12, IC7.13, C?.1
- net at D12.2 (A), IC7.11: now also IC7.9
- net at D12.1 (K), D13.1 (K), R124.1: now also R128.1; no longer R128.2
- net at D13.2 (A): now also IC7.4
- net at IC7.3: now also IC7.5
- net at IC8.10 (+): now also C42.1, C43.1, IC8.1, Pin_B.1 (P1), R114.2
- net TO_PIN_I_NEAR_J150: no longer names the net of J55.2
- net TO_PIN_I_NEAR_J150: now also R128.2, Wire_I1.1 (P1); no longer R128.1
- new net: R?.1, R?.2, RV?.1
- new net: C42.2, IC8.2 (-), R113.2, R114.1
- new net: C43.2, IC8.5 (+), R117.2
- new net: IC8.6 (-), R115.1, R116.2, R?.1, R?.1
- new net: C?.2, IC8.7, R118?.1
- new net: C?.2, IC7.10
- new net: C?.1, D16.1 (K), IC7.8, R?.1
- new net: R123.1, RV4.1
- new net: J?.2 (P2), R?.2
- new net: J?.3 (P3), R?.2
- no-connect marks 1 -> 2
Other:
- note added: "To the sensitivity switch, probably"
- moved on the sheet: C12, C26, C27, C32, C33, D10, D12, D13, D15, D4, D7, D8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
